Commit message: Change grasp object color to red
Gazebo is affected but rviz is not. why?
Also make xterm windows persistent as I wanna debug the errors.
(start script kills all xterms upon enter .. launch.sh does not)

File: optional/kuka_challenge/workspace/catkin_ws/src/rll_planning_project/urdf/grasp_object.urdf.xacro (robot description, xacro)
@@ -26,5 +26,5 @@
     <mu1>1.0</mu1>
     <mu2>1.0</mu2>
-    <material>Gazebo/Blue</material>
+    <material>Gazebo/Red</material>
   </gazebo>
 </robot>

Commit message: Revert marker colors and cosmetics to fix the kuka maze planner
Code runs and object is picked and placed correctly.
I will now work on any path planner algo optimizations.

File: optional/kuka_challenge/workspace/catkin_ws/src/rll_planning_project/urdf/grasp_object.urdf.xacro (robot description, xacro)
@@ -26,5 +26,5 @@
     <mu1>1.0</mu1>
     <mu2>1.0</mu2>
-    <material>Gazebo/Red</material>
+    <material>Gazebo/Blue</material>
   </gazebo>
 </robot>
